Commit message: almost everything working well, documentation not yet complete

File: cob_laser_calibration/objects/cal_obj_pose_verification.urdf (robot description, URDF)
Before this commit: robot calibration_object, 4 links, 3 joints
Links:
- link checkerboard: geometry visual box size=0.4 0.3 0.005
- link cylinder_1: geometry visual cylinder length=0.2 radius=0.09
- link cylinder_2: geometry visual cylinder length=0.2 radius=0.06
- link cylinder_3: geometry visual cylinder length=0.2 radius=0.03
